Commit message: Add files via upload

File: cleaning_robot_assembly_description/urdf/cleaning_robot_assembly.xacro (robot description, xacro)
@@ -6,7 +6,7 @@
 <link name="base_link">
   <inertial>
-    <origin xyz="-0.010230098607375893 -0.0003124840680256018 0.10766281764491467" rpy="0 0 0"/>
-    <mass value="8.266268612843005"/>
-    <inertia ixx="0.111901" iyy="0.101028" izz="0.115277" ixy="-0.003854" iyz="0.0042" ixz="0.003247"/>
+    <origin xyz="-0.010466456463713802 -0.0003168058953017059 0.10831172177775374" rpy="0 0 0"/>
+    <mass value="8.208463592723788"/>
+    <inertia ixx="0.110702" iyy="0.099596" izz="0.113639" ixy="-0.003852" iyz="0.004197" ixz="0.003067"/>
   </inertial>
   <visual>

Commit message: Add files via upload

File: cleaning_robot_assembly_description/urdf/cleaning_robot_assembly.xacro (robot description, xacro)
@@ -6,7 +6,7 @@
 <link name="base_link">
   <inertial>
-    <origin xyz="-0.010466456463713802 -0.0003168058953017059 0.10831172177775374" rpy="0 0 0"/>
-    <mass value="8.208463592723788"/>
-    <inertia ixx="0.110702" iyy="0.099596" izz="0.113639" ixy="-0.003852" iyz="0.004197" ixz="0.003067"/>
+    <origin xyz="-0.010523520290212047 -0.0003161493086687621 0.1081094140538543" rpy="0 0 0"/>
+    <mass value="8.225511131099228"/>
+    <inertia ixx="0.111057" iyy="0.100022" izz="0.114094" ixy="-0.003852" iyz="0.004198" ixz="0.003021"/>
   </inertial>
   <visual>

Commit message: Add files via upload

File: cleaning_robot_assembly_description/urdf/cleaning_robot_assembly.xacro (robot description, xacro)
@@ -24,5 +24,5 @@
   </collision>
 </link>
-<link name="right_wheel_1">
+<link name="right_wheel">
   <inertial>
     <origin xyz="-1.9475303414941916e-15 -0.007842031913982417 1.2323475573339238e-14" rpy="0 0 0"/>
@@ -44,5 +44,5 @@
   </collision>
 </link>
-<link name="left_wheel_1">
+<link name="left_wheel">
   <inertial>
     <origin xyz="2.5866925465521704e-15 0.007842031913982556 1.2288781103819701e-14" rpy="0 0 0"/>
@@ -64,5 +64,5 @@
   </collision>
 </link>
-<link name="ydlidar_1">
+<link name="ydlidar">
   <inertial>
     <origin xyz="0.026706155403509572 0.025000237545982823 0.037701142222791084" rpy="0 0 0"/>
@@ -71,18 +71,18 @@
   </inertial>
   <visual>
+    <origin xyz="0.0 0.0 -0.335" rpy="0 0 0"/>
+    <geometry>
+      <mesh filename="package://cleaning_robot_assembly_description/meshes/ydlidar_1.stl" scale="0.001 0.001 0.001"/>
+    </geometry>
+    <material name="steel_satin"/>
+  </visual>
+  <collision>
     <origin xyz="0.0254 0.025002 -0.293" rpy="0 0 0"/>
     <geometry>
       <mesh filename="package://cleaning_robot_assembly_description/meshes/ydlidar_1.stl" scale="0.001 0.001 0.001"/>
     </geometry>
-    <material name="steel_satin"/>
-  </visual>
-  <collision>
-    <origin xyz="0.0254 0.025002 -0.293" rpy="0 0 0"/>
-    <geometry>
-      <mesh filename="package://cleaning_robot_assembly_description/meshes/ydlidar_1.stl" scale="0.001 0.001 0.001"/>
-    </geometry>
-  </collision>
-</link>
-<link name="fork_lift_1">
+  </collision>
+</link>
+<link name="fork_lift">
   <inertial>
     <origin xyz="0.004496086305917135 0.06235925922763712 -0.023132472112988356" rpy="0 0 0"/>
@@ -95,5 +95,5 @@
       <mesh filename="package://cleaning_robot_assembly_description/meshes/fork_lift_1.stl" scale="0.001 0.001 0.001"/>
     </geometry>
-    <material name="polycarbonate_bronze"/>
+    <material name="steel_satin"/>
   </visual>
   <collision>
@@ -104,5 +104,5 @@
   </collision>
 </link>
-<link name="eef_base_1">
+<link name="eef_base">
   <inertial>
     <origin xyz="0.053928998860087174 0.040021209291948676 -0.009476696298688747" rpy="0 0 0"/>
@@ -124,5 +124,5 @@
   </collision>
 </link>
-<link name="left_finger_1">
+<link name="left_finger">
   <inertial>
     <origin xyz="0.027926963844938285 -0.00977330285299979 0.002500000036867095" rpy="0 0 0"/>
@@ -144,5 +144,5 @@
   </collision>
 </link>
-<link name="right_finger_1">
+<link name="right_finger">
   <inertial>
     <origin xyz="0.02792696384493834 0.009773302853000033 0.002500000037638575" rpy="0 0 0"/>
@@ -164,5 +164,5 @@
   </collision>
 </link>
-<link name="depth_cam_1">
+<link name="depth_cam">
   <inertial>
     <origin xyz="0.008498435151100464 0.022529677339244106 -0.005238954013314812" rpy="0 0 0"/>
@@ -187,48 +187,48 @@
   <origin xyz="0.0 -0.144 0.05" rpy="0 0 0"/>
   <parent link="base_link"/>
-  <child link="right_wheel_1"/>
-  <axis xyz="-0.0 -1.0 0.0"/>
+  <child link="right_wheel"/>
+  <axis xyz="-0.0 1.0 0.0"/>
 </joint>
 <joint name="left_drive" type="continuous">
   <origin xyz="0.0 0.144 0.05" rpy="0 0 0"/>
   <parent link="base_link"/>
-  <child link="left_wheel_1"/>
+  <child link="left_wheel"/>
   <axis xyz="0.0 1.0 0.0"/>
 </joint>
 <joint name="Rigid 3" type="fixed">
-  <origin xyz="-0.0254 -0.025002 0.293" rpy="0 0 0"/>
-  <parent link="base_link"/>
-  <child link="ydlidar_1"/>
+  <origin xyz="-0.0 -0.0 0.335" rpy="0 0 0"/>
+  <parent link="base_link"/>
+  <child link="ydlidar"/>
 </joint>
 <joint name="fork_lift_joint" type="prismatic">
   <origin xyz="0.13885 -0.0797 0.15375" rpy="0 0 0"/>
   <parent link="base_link"/>
-  <child link="fork_lift_1"/>
+  <child link="fork_lift"/>
   <axis xyz="-0.0 0.0 1.0"/>
-  <limit upper="0.0" lower="0.0" effort="100" velocity="100"/>
+  <limit upper="0.125" lower="-0.03" effort="100" velocity="100"/>
 </joint>
 <joint name="Rigid 5" type="fixed">
   <origin xyz="0.007449 0.07895 -0.0239" rpy="0 0 0"/>
-  <parent link="fork_lift_1"/>
-  <child link="eef_base_1"/>
+  <parent link="fork_lift"/>
+  <child link="eef_base"/>
 </joint>
 <joint name="left_pick" type="prismatic">
   <origin xyz="0.066 0.0375 -0.0695" rpy="0 0 0"/>
-  <parent link="eef_base_1"/>
-  <child link="left_finger_1"/>
+  <parent link="eef_base"/>
+  <child link="left_finger"/>
   <axis xyz="-0.0 1.0 0.0"/>
-  <limit upper="0.0" lower="0.0" effort="100" velocity="100"/>
+  <limit upper="0.0125" lower="-0.0125" effort="100" velocity="100"/>
 </joint>
 <joint name="right_pick" type="prismatic">
   <origin xyz="0.066 -0.0375 -0.0695" rpy="0 0 0"/>
-  <parent link="eef_base_1"/>
-  <child link="right_finger_1"/>
+  <parent link="eef_base"/>
+  <child link="right_finger"/>
   <axis xyz="-0.0 1.0 0.0"/>
-  <limit upper="0.0" lower="0.0" effort="100" velocity="100"/>
+  <limit upper="0.0125" lower="-0.0125" effort="100" velocity="100"/>
 </joint>
 <joint name="Rigid 8" type="fixed">
   <origin xyz="0.032345 -0.022492 0.017677" rpy="0 0 0"/>
-  <parent link="eef_base_1"/>
-  <child link="depth_cam_1"/>
+  <parent link="eef_base"/>
+  <child link="depth_cam"/>
 </joint>
 </robot>
