Commit message: Added gazebo plugins and updated urdf

File: cleaning_robot_description/urdf/cleaning_robot.xacro (robot description, xacro)
@@ -18,7 +18,11 @@
   </visual>
   <collision>
-    <origin xyz="0 0 0" rpy="0 0 0"/>
+    <!-- <origin xyz="0 0 0" rpy="0 0 0"/>
     <geometry>
       <mesh filename="package://cleaning_robot_description/meshes/base_link.stl" scale="0.001 0.001 0.001"/>
+    </geometry> -->
+    <origin xyz="0.0 0 0.005" rpy="0 0 0"/>
+    <geometry>
+      <box size="0.35 0.25 0.0085" />
     </geometry>
   </collision>
@@ -88,5 +92,5 @@
   <parent link="base_link"/>
   <child link="right_wheel_1"/>
-  <axis xyz="-0.0 -1.0 0.0"/>
+  <axis xyz="-0.0 1.0 0.0"/>
 </joint>
 <joint name="base2left" type="continuous">

File: cleaning_robot_description/urdf/materials.xacro (robot description, xacro)
@@ -8,5 +8,5 @@
 </material>
 <material name="abs_white">
-  <color rgba="0.9647058823529412 0.9647058823529412 0.9529411764705882 1.0"/>
+  <color rgba="0.2 0.2 0.2 1.0"/>
 </material>
 </robot>

Commit message: reversed lidar joint

File: cleaning_robot_description/urdf/cleaning_robot.xacro (robot description, xacro)
@@ -75,5 +75,5 @@
   </inertial>
   <visual>
-    <origin xyz="0.0 0.0 -0.335" rpy="0 0 0"/>
+    <origin xyz="0.0 0.0 -0.335" rpy="0 0 3.1416"/>
     <geometry>
       <mesh filename="package://cleaning_robot_description/meshes/ydlidar_1.stl" scale="0.001 0.001 0.001"/>
@@ -82,5 +82,5 @@
   </visual>
   <collision>
-    <origin xyz="0.0 0.0 -0.335" rpy="0 0 0"/>
+    <origin xyz="0.0 0.0 -0.335" rpy="0 0 3.1416"/>
     <geometry>
       <mesh filename="package://cleaning_robot_description/meshes/ydlidar_1.stl" scale="0.001 0.001 0.001"/>
@@ -101,5 +101,5 @@
 </joint>
 <joint name="base2lidar" type="fixed">
-  <origin xyz="-0.0 -0.0 0.335" rpy="0 0 0"/>
+  <origin xyz="-0.0 -0.0 0.335" rpy="0 0 3.1416"/>
   <parent link="base_link"/>
   <child link="ydlidar_1"/>
